File: hardware/STM32H745_Ballistic_Corrector.kicad_pcb (KiCad board)
At the start: 4 copper layers, 80 x 60 mm, 52 parts, among them J1 12V_IN, J2 UART_DBG, J3 SWD, J4 SENSOR_14P, J5 USB_MINI_B, SW1 BOOT0, U1 STM32H745ZIT6, U10 MCP9808, U11 BMP390, U12 LDO_1V8_200mA, U2 TPS62133A, U3 LDO_3V3_500mA, U4 ICM-20689, U5 VL53L0X, U6 W25Q128JV, U7 AT24C256C, U8 CP2102N, Y1 8MHz

Commit message: PCB step 7: power routing complete; fix D1/J1 pad overlap (placement)
- Placement blind spot found: the courtyard checker compares F.Fab bodies,
  not courtyards, so D1's SMA pads silently overlapped J1's sleeve TH pad.
  Power row shifted east (D1->74, U2->78.5, L1->84, C2->89, U3->96,
  C14->102, U12->107.5, C15->112); checker limitation logged as tech debt
- New nets: PWR_12V_RAW (pre-diode) and PWR_SW (buck switch node), bound
  in placement (J1.1, D1.1/D1.2, U2 pin5, L1.1)
- Power routing: raw 12V arc around J1 sleeve; buck VIN riser + EN tied
  via a short B.Cu hop (F.Cu strap cannot clear the 0.95mm pin field);
  0.8mm SW node; 5V rail L1->C2->via into the In2 5V pour; LDO feeds
  from the pour; 3V3 drops (U3 pin2 + tab, C14, TP3 detour x119.5) into
  the In2 3V3 pour; local 1V8 spine U12->C15->TP4; GND drops throughout
- Audit iterations: 5 -> 0 violations. Totals: 216 segments, 100 vias,
  QSPI skew still 0.01mm, courtyard/body check PASS
- Deferred: TP1 12V tie (B.Cu power distribution pass in KiCad)

Co-Authored-By: Claude Fable 5 <noreply@anthropic.com>
Claude-Session: https://claude.ai/code/session_01WTnjtLhvvQkSSzjNBr8Vvw
Parts:
- moved D1 3.50 mm to (74.0, 56.5)
- moved C14 2.00 mm to (102.0, 56.5)
- moved C2 2.00 mm to (89.0, 56.5)
- moved L1 2.00 mm to (84.0, 56.5)
- moved U2 2.00 mm to (78.5, 56.5)
- moved U3 2.00 mm to (96.0, 56.5)
- moved U12 1.50 mm to (107.5, 56.5)
- moved C15 1.00 mm to (112.0, 56.5)
Connections:
- D1 pad 1: (no net) -> PWR_12V_RAW
- J1 pad 1: VCC_12V -> PWR_12V_RAW
- L1 pad 1: (no net) -> PWR_SW
- U2 pad 5: (no net) -> PWR_SW
Routing:
- net VCC_3V3: track 46.6 -> 79.0 mm, vias 27 -> 31
- net VCC_1V8: track 0.00 -> 21.8 mm
- net PWR_12V_RAW: track 0.00 -> 14.6 mm
- net GND: track 38.4 -> 48.7 mm, vias 26 -> 32
- net VCC_12V: track 0.00 -> 9.10 mm, vias 0 -> 2
- net PWR_SW: track 0.00 -> 8.45 mm
- net VCC_5V: track 1.20 -> 7.75 mm, vias 1 -> 4
Changed lines of the file:
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@@
   (net 22 "NRST")
   (net 23 "BOOT0")
+  (net 24 "PWR_SW")
+  (net 25 "PWR_12V_RAW")
   ;; ------------------------------------------------------------------
   ;; Board outline: 80 x 60 mm, origin (50,50) .. (130,110), R2 corners
@@
     (fp_rect (start -4.5 -5.5) (end 4.5 5.5) (stroke (width 0.12) (type solid)) (fill none) (layer "F.Fab"))
     (fp_rect (start -5 -6) (end 5 6) (stroke (width 0.05) (type solid)) (fill none) (layer "F.CrtYd"))
-    (pad "1" thru_hole rect (at 0 0) (size 3 3) (drill 1.6) (layers "*.Cu" "*.Mask") (net 5 "VCC_12V"))
+    (pad "1" thru_hole rect (at 0 0) (size 3 3) (drill 1.6) (layers "*.Cu" "*.Mask") (net 25 "PWR_12V_RAW"))
     (pad "2" thru_hole circle (at 6.1 0) (size 3 3) (drill 1.6) (layers "*.Cu" "*.Mask") (net 1 "GND"))
     (pad "3" thru_hole circle (at 3 4.6) (size 3 3) (drill 1.6) (layers "*.Cu" "*.Mask") (net 1 "GND"))
   )
-  (footprint "Diode_SMD:D_SMA" (layer "F.Cu") (at 70.5 56.5 0)
+  (footprint "Diode_SMD:D_SMA" (layer "F.Cu") (at 74 56.5 0)
     (descr "Reverse polarity Schottky")
     (attr smd)
@@
     (fp_rect (start -2.9 -0.9) (end 2.9 0.9) (stroke (width 0.12) (type solid)) (fill none) (layer "F.Fab"))
     (fp_rect (start -3.4 -1.4) (end 3.4 1.4) (stroke (width 0.05) (type solid)) (fill none) (layer "F.CrtYd"))
-    (pad "1" smd roundrect (at -2.15 0) (size 1.5 1.8) (layers "F.Cu" "F.Paste" "F.Mask") (roundrect_rratio 0.25))
+    (pad "1" smd roundrect (at -2.15 0) (size 1.5 1.8) (layers "F.Cu" "F.Paste" "F.Mask") (roundrect_rratio 0.25) (net 25 "PWR_12V_RAW"))
     (pad "2" smd roundrect (at 2.15 0) (size 1.5 1.8) (layers "F.Cu" "F.Paste" "F.Mask") (roundrect_rratio 0.25) (net 5 "VCC_12V"))
   )
-  (footprint "Package_TO_SOT_SMD:SOT-23-5" (layer "F.Cu") (at 76.5 56.5 0)
+  (footprint "Package_TO_SOT_SMD:SOT-23-5" (layer "F.Cu") (at 78.5 56.5 0)
     (descr "Buck 12V->5V; VERIFY package vs ordered part variant")
     (attr smd)
@@
     (pad "3" smd roundrect (at 0.95 1.3) (size 0.6 1.2) (layers "F.Cu" "F.Paste" "F.Mask") (roundrect_rratio 0.25) (net 5 "VCC_12V"))
     (pad "4" smd roundrect (at 0.95 -1.3) (size 0.6 1.2) (layers "F.Cu" "F.Paste" "F.Mask") (roundrect_rratio 0.25))
-    (pad "5" smd roundrect (at -0.95 -1.3) (size 0.6 1.2) (layers "F.Cu" "F.Paste" "F.Mask") (roundrect_rratio 0.25))
-  )
-  (footprint "Inductor_SMD:L_4x4mm" (layer "F.Cu") (at 82 56.5 0)
+    (pad "5" smd roundrect (at -0.95 -1.3) (size 0.6 1.2) (layers "F.Cu" "F.Paste" "F.Mask") (roundrect_rratio 0.25) (net 24 "PWR_SW"))
+  )
+  (footprint "Inductor_SMD:L_4x4mm" (layer "F.Cu") (at 84 56.5 0)
     (descr "Buck inductor")
     (attr smd)
@@
     (fp_rect (start -2.3 -1.8) (end 2.3 1.8) (stroke (width 0.12) (type solid)) (fill none) (layer "F.Fab"))
     (fp_rect (start -2.8 -2.3) (end 2.8 2.3) (stroke (width 0.05) (type solid)) (fill none) (layer "F.CrtYd"))
-    (pad "1" smd roundrect (at -1.7 0) (size 1.2 3.6) (layers "F.Cu" "F.Paste" "F.Mask") (roundrect_rratio 0.25))
+    (pad "1" smd roundrect (at -1.7 0) (size 1.2 3.6) (layers "F.Cu" "F.Paste" "F.Mask") (roundrect_rratio 0.25) (net 24 "PWR_SW"))
     (pad "2" smd roundrect (at 1.7 0) (size 1.2 3.6) (layers "F.Cu" "F.Paste" "F.Mask") (roundrect_rratio 0.25) (net 4 "VCC_5V"))
   )
-  (footprint "Capacitor_SMD:C_0805" (layer "F.Cu") (at 87 56.5 0)
+  (footprint "Capacitor_SMD:C_0805" (layer "F.Cu") (at 89 56.5 0)
     (descr "5V bulk")
     (attr smd)
@@
     (pad "2" smd roundrect (at 0.95 0) (size 1 1.3) (layers "F.Cu" "F.Paste" "F.Mask") (roundrect_rratio 0.25) (net 1 "GND"))
   )
-  (footprint "Package_TO_SOT_SMD:SOT-223" (layer "F.Cu") (at 94 56.5 0)
+  (footprint "Package_TO_SOT_SMD:SOT-223" (layer "F.Cu") (at 96 56.5 0)
     (descr "3V3 LDO")
     (attr smd)
@@
     (pad "4" smd roundrect (at 0 -3.2) (size 3.6 2.2) (layers "F.Cu" "F.Paste" "F.Mask") (roundrect_rratio 0.25) (net 2 "VCC_3V3"))
   )
-  (footprint "Capacitor_SMD:C_0805" (layer "F.Cu") (at 100 56.5 0)
+  (footprint "Capacitor_SMD:C_0805" (layer "F.Cu") (at 102 56.5 0)
     (descr "3V3 bulk")
     (attr smd)
@@
     (pad "2" smd roundrect (at 0.95 0) (size 1 1.3) (layers "F.Cu" "F.Paste" "F.Mask") (roundrect_rratio 0.25) (net 1 "GND"))
   )
-  (footprint "Package_TO_SOT_SMD:SOT-23-5" (layer "F.Cu") (at 106 56.5 0)
+  (footprint "Package_TO_SOT_SMD:SOT-23-5" (layer "F.Cu") (at 107.5 56.5 0)
     (descr "1V8 LDO")
     (attr smd)
@@
     (pad "5" smd roundrect (at -0.95 -1.3) (size 0.6 1.2) (layers "F.Cu" "F.Paste" "F.Mask") (roundrect_rratio 0.25) (net 3 "VCC_1V8"))
   )
-  (footprint "Capacitor_SMD:C_0805" (layer "F.Cu") (at 111 56.5 0)
+  (footprint "Capacitor_SMD:C_0805" (layer "F.Cu") (at 112 56.5 0)
     (descr "1V8 bulk")
     (attr smd)
@@
   (segment (start 57.2 90) (end 57.2 82) (width 0.2) (layer "F.Cu") (net 21))
   (segment (start 57.2 82) (end 55.5 82) (width 0.2) (layer "F.Cu") (net 21))
+  (segment (start 63 56.5) (end 63 53.6) (width 1) (layer "F.Cu") (net 25))
+  (segment (start 63 53.6) (end 71.85 53.6) (width 1) (layer "F.Cu") (net 25))
+  (segment (start 71.85 53.6) (end 71.85 56.5) (width 1) (layer "F.Cu") (net 25))
+  (segment (start 76.15 56.5) (end 77.55 56.5) (width 0.5) (layer "F.Cu") (net 5))
+  (segment (start 77.55 56.5) (end 77.55 57.8) (width 0.5) (layer "F.Cu") (net 5))
+  (segment (start 79.45 57.8) (end 79.45 58.7) (width 0.3) (layer "F.Cu") (net 5))
+  (segment (start 79.45 58.7) (end 76.15 58.7) (width 0.3) (layer "B.Cu") (net 5))
+  (segment (start 76.15 58.7) (end 76.15 57.4) (width 0.3) (layer "B.Cu") (net 5))
+  (segment (start 76.15 57.4) (end 76.15 56.5) (width 0.3) (layer "F.Cu") (net 5))
+  (segment (start 77.55 55.2) (end 77.55 54) (width 0.8) (layer "F.Cu") (net 24))
+  (segment (start 77.55 54) (end 82.3 54) (width 0.8) (layer "F.Cu") (net 24))
+  (segment (start 82.3 54) (end 82.3 56.5) (width 0.8) (layer "F.Cu") (net 24))
+  (segment (start 85.7 56.5) (end 88.05 56.5) (width 1) (layer "F.Cu") (net 4))
+  (segment (start 88.05 56.5) (end 88.05 55) (width 0.8) (layer "F.Cu") (net 4))
+  (segment (start 89.95 56.5) (end 89.95 55) (width 0.8) (layer "F.Cu") (net 1))
+  (segment (start 98.3 59.7) (end 99.6 59.7) (width 0.8) (layer "F.Cu") (net 4))
+  (segment (start 106.55 57.8) (end 106.55 59.2) (width 0.5) (layer "F.Cu") (net 4))
+  (segment (start 96 59.7) (end 96 62.8) (width 0.8) (layer "F.Cu") (net 2))
+  (segment (start 96 53.3) (end 92.3 53.3) (width 0.8) (layer "F.Cu") (net 2))
+  (segment (start 92.3 53.3) (end 92.3 62.8) (width 0.8) (layer "F.Cu") (net 2))
+  (segment (start 93.7 59.7) (end 93.7 61.9) (width 0.5) (layer "F.Cu") (net 1))
+  (segment (start 101.05 56.5) (end 101.05 62.8) (width 0.5) (layer "F.Cu") (net 2))
+  (segment (start 102.95 56.5) (end 102.95 55) (width 0.5) (layer "F.Cu") (net 1))
+  (segment (start 106.55 55.2) (end 106.55 53.3) (width 0.5) (layer "F.Cu") (net 3))
+  (segment (start 106.55 53.3) (end 116.5 53.3) (width 0.5) (layer "F.Cu") (net 3))
+  (segment (start 116.5 53.3) (end 116.5 58.5) (width 0.5) (layer "F.Cu") (net 3))
+  (segment (start 116.5 58.5) (end 115 58.5) (width 0.5) (layer "F.Cu") (net 3))
+  (segment (start 111.05 53.3) (end 111.05 56.5) (width 0.5) (layer "F.Cu") (net 3))
+  (segment (start 112.95 56.5) (end 112.95 55) (width 0.5) (layer "F.Cu") (net 1))
+  (segment (start 107.5 57.8) (end 107.5 59.3) (width 0.5) (layer "F.Cu") (net 1))
+  (segment (start 78.5 57.8) (end 78.5 59.9) (width 0.5) (layer "F.Cu") (net 1))
+  (segment (start 121 54.5) (end 119.5 54.5) (width 0.5) (layer "F.Cu") (net 2))
+  (segment (start 119.5 54.5) (end 119.5 62.8) (width 0.5) (layer "F.Cu") (net 2))
   (via (at 102.45 83.8) (size 0.6) (drill 0.3) (layers "F.Cu" "B.Cu") (net 7))
   (via (at 117.7 74.6) (size 0.6) (drill 0.3) (layers "F.Cu" "B.Cu") (net 7))
@@
   (via (at 93.9 99.2) (size 0.6) (drill 0.3) (layers "F.Cu" "B.Cu") (net 17))
   (via (at 115.2 87.905) (size 0.6) (drill 0.3) (layers "F.Cu" "B.Cu") (net 17))
+  (via (at 79.45 58.7) (size 0.6) (drill 0.3) (layers "F.Cu" "B.Cu") (net 5))
+  (via (at 76.15 57.4) (size 0.6) (drill 0.3) (layers "F.Cu" "B.Cu") (net 5))
+  (via (at 88.05 55) (size 0.6) (drill 0.3) (layers "F.Cu" "B.Cu") (net 4))
+  (via (at 89.95 55) (size 0.6) (drill 0.3) (layers "F.Cu" "B.Cu") (net 1))
+  (via (at 99.6 59.7) (size 0.6) (drill 0.3) (layers "F.Cu" "B.Cu") (net 4))
+  (via (at 106.55 59.2) (size 0.6) (drill 0.3) (layers "F.Cu" "B.Cu") (net 4))
+  (via (at 96 62.8) (size 0.6) (drill 0.3) (layers "F.Cu" "B.Cu") (net 2))
+  (via (at 92.3 62.8) (size 0.6) (drill 0.3) (layers "F.Cu" "B.Cu") (net 2))
+  (via (at 93.7 61.9) (size 0.6) (drill 0.3) (layers "F.Cu" "B.Cu") (net 1))
+  (via (at 101.05 62.8) (size 0.6) (drill 0.3) (layers "F.Cu" "B.Cu") (net 2))
+  (via (at 102.95 55) (size 0.6) (drill 0.3) (layers "F.Cu" "B.Cu") (net 1))
+  (via (at 112.95 55) (size 0.6) (drill 0.3) (layers "F.Cu" "B.Cu") (net 1))
+  (via (at 107.5 59.3) (size 0.6) (drill 0.3) (layers "F.Cu" "B.Cu") (net 1))
+  (via (at 78.5 59.9) (size 0.6) (drill 0.3) (layers "F.Cu" "B.Cu") (net 1))
+  (via (at 119.5 62.8) (size 0.6) (drill 0.3) (layers "F.Cu" "B.Cu") (net 2))
   ;; END GENERATED ROUTING
 )
